File: circuits/3v3_to_cv.kicad_sch (KiCad schematic)
At the start: 17 parts, among them U2 TL074CDT, U3 LM324

Commit message: fixed circuits, added 74HC589 symbol
Connections:
- net CV_3V3_1: now also U2.3 (+); no longer U2.2 (-)
- net CV_3V3_2: now also U2.5 (+); no longer U2.6 (-)
- net CV_3V3_3: now also U2.10 (+); no longer U2.9 (-)
- net CV_3V3_4: now also U2.12 (+); no longer U2.13 (-)
- net at C2.2, R19.2, R21.2: now also U2.2 (-); no longer U2.3 (+)
- net at C3.2, R20.2, R22.2: now also U2.9 (-); no longer U2.10 (+)
- net at C4.2, R23.2, R25.2: now also U2.6 (-); no longer U2.5 (+)
- net at C5.2, R24.2, R26.2: now also U2.13 (-); no longer U2.12 (+)
Changed lines of the file:
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@@
     (pin "1")
   )
-  (symbol (lib_id "Device:Opamp_Quad_Generic") (at 146.05 86.36 0) (unit 1)
-    (in_bom yes) (on_board yes)
-    (property "Reference" "U2" (id 0) (at 147.32 77.47 0))
-    (property "Value" "TL074CDT" (id 1) (at 147.32 80.01 0))
+  (symbol (lib_id "Device:Opamp_Quad_Generic") (at 146.05 86.36 0) (mirror x) (unit 1)
+    (in_bom yes) (on_board yes)
+    (property "Reference" "U2" (id 0) (at 147.32 95.25 0))
+    (property "Value" "TL074CDT" (id 1) (at 147.32 92.71 0))
     (property "Footprint" "" (id 2) (at 146.05 86.36 0)
       (effects (font (size 1.27 1.27)) hide)
@@
     (pin "2")
   )
-  (symbol (lib_id "Device:Opamp_Quad_Generic") (at 146.05 142.24 0) (unit 3)
-    (in_bom yes) (on_board yes)
-    (property "Reference" "U2" (id 0) (at 147.32 133.35 0))
-    (property "Value" "TL074CDT" (id 1) (at 147.32 135.89 0))
+  (symbol (lib_id "Device:Opamp_Quad_Generic") (at 146.05 142.24 0) (mirror x) (unit 3)
+    (in_bom yes) (on_board yes)
+    (property "Reference" "U2" (id 0) (at 147.32 151.13 0))
+    (property "Value" "TL074CDT" (id 1) (at 147.32 148.59 0))
     (property "Footprint" "" (id 2) (at 146.05 142.24 0)
       (effects (font (size 1.27 1.27)) hide)
@@
     (pin "2")
   )
-  (symbol (lib_id "Device:Opamp_Quad_Generic") (at 233.68 83.82 0) (unit 2)
-    (in_bom yes) (on_board yes)
-    (property "Reference" "U2" (id 0) (at 234.95 74.93 0))
-    (property "Value" "TL074CDT" (id 1) (at 234.95 77.47 0))
+  (symbol (lib_id "Device:Opamp_Quad_Generic") (at 233.68 83.82 0) (mirror x) (unit 2)
+    (in_bom yes) (on_board yes)
+    (property "Reference" "U2" (id 0) (at 234.95 92.71 0))
+    (property "Value" "TL074CDT" (id 1) (at 234.95 90.17 0))
     (property "Footprint" "" (id 2) (at 233.68 83.82 0)
       (effects (font (size 1.27 1.27)) hide)
@@
     (pin "2")
   )
-  (symbol (lib_id "Device:Opamp_Quad_Generic") (at 233.68 139.7 0) (unit 4)
-    (in_bom yes) (on_board yes)
-    (property "Reference" "U2" (id 0) (at 234.95 130.81 0))
-    (property "Value" "TL074CDT" (id 1) (at 234.95 133.35 0))
+  (symbol (lib_id "Device:Opamp_Quad_Generic") (at 233.68 139.7 0) (mirror x) (unit 4)
+    (in_bom yes) (on_board yes)
+    (property "Reference" "U2" (id 0) (at 234.95 148.59 0))
+    (property "Value" "TL074CDT" (id 1) (at 234.95 146.05 0))
     (property "Footprint" "" (id 2) (at 233.68 139.7 0)
       (effects (font (size 1.27 1.27)) hide)
